File: keyboard.kicad_pcb (KiCad board)
At the start: 2 copper layers, 116.7 x 27.8 mm, 24 parts, among them SW1 SW_Push, U1 ATmega32U4-A, Y1 16MHz

Commit message: e
Parts:
- moved R1 22.8 mm to (53.8, 98.8)
Routing:
- net +5V: track 10.3 -> 100.5 mm, vias 2 -> 7
- net GND: track 49.9 -> 134.7 mm, vias 0 -> 2
- net ROW0: track 0.00 -> 63.8 mm
- net VCC: track 0.00 -> 10.0 mm, vias 0 -> 2
- net Net-(D3-Pad2): track 0.00 -> 8.64 mm
- net Net-(D2-Pad2): track 0.00 -> 8.64 mm
- net Net-(D1-Pad2): track 0.00 -> 8.64 mm
- net Net-(D4-Pad2): track 0.00 -> 8.64 mm
- net Net-(C2-Pad2): track 2.91 -> 10.1 mm
- net Net-(R1-Pad2): track 14.2 -> 19.1 mm
- net Net-(C1-Pad2): track 2.97 -> 7.60 mm
Other:
- board text added: "Made by HoosierTransfer"

Commit message: k
Connections:
- U1 pad 11: COL3 -> unconnected-(U1-Pad11)
- U1 pad 27: ROW0 -> unconnected-(U1-Pad27)
- U1 pad 28: COL2 -> unconnected-(U1-Pad28)
- U1 pad 29: COL1 -> unconnected-(U1-Pad29)
- U1 pad 30: COL0 -> unconnected-(U1-Pad30)
Routing:
- net unconnected-(USB1-Pad6): track 0.00 -> 16.3 mm
- net +5V: track 100.5 -> 113.9 mm
- net GND: track 134.7 -> 142.4 mm

Commit message: f
Parts:
- moved C2 0.53 mm to (60.0, 98.7)
- moved C1 0.47 mm to (69.0, 98.8)
Connections:
- U1 pad 25: unconnected-(U1-Pad25) -> ROW0
- U1 pad 26: unconnected-(U1-Pad26) -> COL3
- U1 pad 27: unconnected-(U1-Pad27) -> COL2
- U1 pad 28: unconnected-(U1-Pad28) -> COL1
- U1 pad 29: unconnected-(U1-Pad29) -> COL0
Routing:
- net COL3: track 0.00 -> 86.4 mm, vias 0 -> 2
- net COL2: track 0.00 -> 65.0 mm, vias 0 -> 4
- net COL1: track 0.00 -> 40.3 mm, vias 0 -> 2
- net ROW0: track 63.8 -> 90.7 mm, vias 0 -> 2
- net COL0: track 0.00 -> 14.7 mm, vias 0 -> 2
- net GND: track 142.4 -> 141.1 mm
- added copper zone on F.Cu, net GND
Other:
- board text added: "4k Keyboard"

Commit message: f
Parts:
- D1, D2, D4: value SOD-123 -> 1N4148W-TP
- moved F1 22.3 mm to (64.5, 80.0), turned to 0 degrees
- moved R2 3.83 mm to (49.1, 88.8), turned to 0 degrees
- moved C4 1.90 mm to (55.4, 84.4)
- moved R1 1.90 mm to (53.4, 100.7)
- moved Y1 1.90 mm to (64.1, 100.6)
- moved C3 1.90 mm to (54.3, 91.5)
- moved D4 1.90 mm to (153.6, 90.8)
- moved MX4 1.90 mm to (145.6, 90.8)
- moved C1 1.90 mm to (68.6, 100.6)
- moved C5 1.90 mm to (72.8, 96.3)
- moved C6 1.90 mm to (69.0, 79.9)
- moved C7 1.90 mm to (60.1, 79.9)
- moved D1 1.90 mm to (96.4, 90.8)
- moved D2 1.90 mm to (115.5, 90.8)
- moved MX1 1.90 mm to (88.5, 90.8)
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Connections:
- net Net-(R2-Pad2) renamed D0+
- net Net-(R3-Pad2) renamed D0-
Routing:
- net +5V: track 113.8 -> 136.8 mm
- net VCC: track 10.0 -> 24.7 mm, vias 2 -> 0
- net D0+: track 13.4 -> 9.20 mm
- net D+: track 4.44 -> 8.63 mm
- net GND: track 141.1 -> 138.9 mm
- net D-: track 4.44 -> 6.14 mm
- net D0-: track 10.5 -> 9.18 mm
Other:
- board size 116.7 x 27.8 mm -> 117.5 x 31.8 mm
